File: BSPD/BSPD.kicad_sch (KiCad schematic)
At the start: 46 parts, among them J1 Conn_01x02_Socket, J2 Conn_01x02_Socket, J3 Conn_01x02_Socket, K1 Fujitsu_FTR-LYCA005x, Q1 PMOS, Q2 PMOS, Q3 NMOS, U1 LM393, U2 CD4081BM, U3 LM393, U4 CD4043BD, U5 CD4011BM, U6 LM393

Commit message: Added upto date files.
Extra circuit added for overvoltage as well as reverse voltage protection.
Parts:
- added D4, D5: LED, symbol Device:LED
- added D6, D7: D_Zener, symbol Device:D_Zener
- added Q4, Q5, Q6: PMOS, symbol Simulation_SPICE:PMOS
- added R13, R14, R17, R2, R6: R, symbol Device:R
- added R3, R5: 100k, symbol Device:R
Connections:
- net GLV+: now also U1.4 (V-), U3.8 (V+), Q4.1 (D), Q6.1 (D), R3.1; no longer D3.1 (K), U1.8 (V+), U3.4 (V-)
- net GLV-: now also U1.8 (V+), U3.4 (V-), D6.2 (A), R13.2, R17.2, R2.1, R6.1; no longer D3.2 (A), U1.4 (V-), U3.8 (V+)
- net Q_output: now also R5.2
- new net: D4.2 (A), R2.2, R3.2
- new net: D3.1 (K), D7.1 (K), Q4.3 (S), Q5.3 (S), Q6.3 (S), R14.1
- new net: D7.2 (A), Q5.1 (D), Q6.2 (G), R17.1
- new net: D4.1 (K), R5.1, R6.2
- new net: D6.1 (K), Q5.2 (G), R14.2
- new net: D3.2 (A), Q4.2 (G), R13.1
Other:
- note added: "TODO: 1) Look into waveforms of the inputs and outputs of the SR Latch. 2) Change the current relay with a TI one. 3) To replace the resistor and capcitor values after a simulation. For timing c and r's, use laplace transformation for both charging and discharging. For the "schmitt triggers", the link below : https://www.youtube.com/watch?v=c59My7goiAE 4) Replace NMOS and PMOS placeholder symbols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"
- note added: "This is just a experimental setup to prevent overvoltage and reverse voltage from destroying the components. Better implemented in the Power distribution board. Because : 1) Cheaper as less components required than implementing in each LV board. 2) Common power to all, this can help in removing headaches of debugging if something goes wrong. Circuit working : https://electronics.stackexchange.com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"
- note removed: "TODO: 1) There is no need to be worried about the invalid state of the SR Latch, as the state of both SET and RESET being HIGH at the same time is highly unlikely. Look into waveforms of the inputs and outputs of the SR Latch. 2) Change the current relay with a TI one. 3) To replace the resistor and capcitor values after a simulation. 4) Replace NMOS and PMOS placeholder symbols with actual ones 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"
- company: (none) -> Ashwa Mobility Foundation
- title: (none) -> Brake System Plausibility Device according to FSG 2025
- moved on the sheet: J1, J2, J3

Commit message: Add files via upload
Parts:
- removed U2: CD4081BM, D14, symbol CD4081B:CD4081BM
- removed U4: CD4043BD, D16, symbol CD4043BD:CD4043BD
- added C4: C, symbol Device:C
- added D8: LED, symbol Device:LED
- added R18, R32: R, symbol Device:R
- added U2: CD4081BM, D14, symbol CD4081BM:CD4081BM
- added unit 5 of U5
- added unit 3 of U5
- added unit 2 of U5
- added unit 4 of U5
Connections:
- net 10s_comparator_output: now also D8.2 (A), R32.2
- net 500ms_comparator_output: now also D5.2 (A), R18.2, U2.5 (C)
- net GLV+: now also C4.1, U2.14 (VDD), U5.14 (VDD); no longer U5.14 (VDD)
- net GLV-: now also D5.1 (K), C4.2, D8.1 (K), R18.1, R32.1, U2.7 (VSS), U5.7 (VSS); no longer U5.7 (VSS)
- net Implausiblity: now also U2.4 (K)
- net Plausibility: now also U2.3 (J)
- net Plausibility_NOT: now also U5.3 (J), U2.6 (D); no longer U5.9 (J)
- net Brake_pressure_sensor_comparator_output: no longer names the net of R10.2, R7.2, U1.7
- net Brake_pressure_sensor_comparator_output: now also U2.2 (B)
- net Current_sensor_comparator_output: no longer names the net of R8.2, R9.1, U1.1
- net Current_sensor_comparator_output: now also U2.1 (A)
- net Q_output: no longer names the net of R23.1, R5.2
Other:
- note added: "Redundant Compoents"
- note removed: "AND GATE"
- note removed: "AND GATE, NAND GATE & SR LATCH (CD 4000 series)"
- note removed: "NAND GATE"
- note removed: "SR LATCH"
- moved on the sheet: C1, C2, C3, D1, D2, D4, D5, J1, J2, J3, K1, Q1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
